Commit message: Update ur3.ros2_control.xacro

File: ur3_description/urdf/ur3.ros2_control.xacro (robot description, xacro)
@@ -3,5 +3,49 @@
   <xacro:macro name="ur3_ros2_control" params="name prefix">
     <ros2_control name="${name}" type="system">
-      <!-- add controller info here -->
+      <hardware>
+        <plugin>ign_ros2_control/IgnitionSystem</plugin>
+      </hardware>
+      <joint name="${prefix}shoulder_pan_joint">
+        <command_interface name="position"/>
+        <state_interface name="position"/>
+        <state_interface name="velocity"/>
+        <param name="min_position">-3.14159265359</param>
+        <param name="max_position">3.14159265359</param>
+      </joint>
+      <joint name="${prefix}shoulder_lift_joint">
+        <command_interface name="position"/>
+        <state_interface name="position"/>
+        <state_interface name="velocity"/>
+        <param name="min_position">-3.14159265359</param>
+        <param name="max_position">3.14159265359</param>
+      </joint>
+      <joint name="${prefix}elbow_joint">
+        <command_interface name="position"/>
+        <state_interface name="position"/>
+        <state_interface name="velocity"/>
+        <param name="min_position">-1.57079632679</param>
+        <param name="max_position">1.57079632679</param>
+      </joint>
+      <joint name="${prefix}wrist_1_joint">
+        <command_interface name="position"/>
+        <state_interface name="position"/>
+        <state_interface name="velocity"/>
+        <param name="min_position">-6.28318530718</param>
+        <param name="max_position">6.28318530718</param>
+      </joint>
+      <joint name="${prefix}wrist_2_joint">
+        <command_interface name="position"/>
+        <state_interface name="position"/>
+        <state_interface name="velocity"/>
+        <param name="min_position">-6.28318530718</param>
+        <param name="max_position">6.28318530718</param>
+      </joint>
+      <joint name="${prefix}wrist_3_joint">
+        <command_interface name="position"/>
+        <state_interface name="position"/>
+        <state_interface name="velocity"/>
+        <param name="min_position">-6.28318530718</param>
+        <param name="max_position">6.28318530718</param>
+      </joint>
     </ros2_control>
   </xacro:macro>
