Commit message: Added ros2 controller

File: ur3_description/urdf/ur3.gazebo.xacro (robot description, xacro)
@@ -4,3 +4,9 @@
     <!-- add plugin info here -->
   </gazebo>
+  <gazebo>
+    <!-- Joint state publisher -->
+    <plugin filename="gz_ros2_control-system" name="gz_ros2_control::GazeboSimROS2ControlPlugin">
+      <parameters>$(find ur3_description)/config/ur3_controllers.yaml</parameters>
+    </plugin>
+  </gazebo>
 </robot>

File: ur3_description/urdf/ur3.ros2_control.xacro (robot description, xacro)
@@ -1,50 +1,69 @@
 <?xml version="1.0"?>
 <robot xmlns:xacro="http://ros.org/wiki/xacro">
-  <xacro:macro name="ur3_ros2_control" params="name prefix">
+  <xacro:macro name="ur3_ros2_control" params="name prefix
+        initial_positions:=${dict(shoulder_pan_joint=0.0,shoulder_lift_joint=-1.57,elbow_joint=0.0,wrist_1_joint=-1.57,wrist_2_joint=0.0,wrist_3_joint=0.0)}">
     <ros2_control name="${name}" type="system">
       <hardware>
-        <plugin>ign_ros2_control/IgnitionSystem</plugin>
+        <plugin>gz_ros2_control/GazeboSimSystem</plugin>
       </hardware>
       <joint name="${prefix}shoulder_pan_joint">
         <command_interface name="position"/>
-        <state_interface name="position"/>
+        <command_interface name="velocity"/>
+        <state_interface name="position">
+          <!-- initial position for the FakeSystem and simulation -->
+          <param name="initial_value">${initial_positions['shoulder_pan_joint']}</param>
+        </state_interface>
         <state_interface name="velocity"/>
-        <param name="min_position">-3.14159265359</param>
-        <param name="max_position">3.14159265359</param>
+        <state_interface name="effort"/>
       </joint>
       <joint name="${prefix}shoulder_lift_joint">
         <command_interface name="position"/>
-        <state_interface name="position"/>
+        <command_interface name="velocity"/>
+        <state_interface name="position">
+          <!-- initial position for the FakeSystem and simulation -->
+          <param name="initial_value">${initial_positions['shoulder_lift_joint']}</param>
+        </state_interface>
         <state_interface name="velocity"/>
-        <param name="min_position">-3.14159265359</param>
-        <param name="max_position">3.14159265359</param>
+        <state_interface name="effort"/>
       </joint>
       <joint name="${prefix}elbow_joint">
         <command_interface name="position"/>
-        <state_interface name="position"/>
+        <command_interface name="velocity"/>
+        <state_interface name="position">
+          <!-- initial position for the FakeSystem and simulation -->
+          <param name="initial_value">${initial_positions['elbow_joint']}</param>
+        </state_interface>
         <state_interface name="velocity"/>
-        <param name="min_position">-1.57079632679</param>
-        <param name="max_position">1.57079632679</param>
+        <state_interface name="effort"/>
       </joint>
       <joint name="${prefix}wrist_1_joint">
         <command_interface name="position"/>
-        <state_interface name="position"/>
+        <command_interface name="velocity"/>
+        <state_interface name="position">
+          <!-- initial position for the FakeSystem and simulation -->
+          <param name="initial_value">${initial_positions['wrist_1_joint']}</param>
+        </state_interface>
         <state_interface name="velocity"/>
-        <param name="min_position">-6.28318530718</param>
-        <param name="max_position">6.28318530718</param>
+        <state_interface name="effort"/>
       </joint>
       <joint name="${prefix}wrist_2_joint">
         <command_interface name="position"/>
-        <state_interface name="position"/>
+        <command_interface name="velocity"/>
+        <state_interface name="position">
+          <!-- initial position for the FakeSystem and simulation -->
+          <param name="initial_value">${initial_positions['wrist_2_joint']}</param>
+        </state_interface>
         <state_interface name="velocity"/>
-        <param name="min_position">-6.28318530718</param>
-        <param name="max_position">6.28318530718</param>
+        <state_interface name="effort"/>
       </joint>
       <joint name="${prefix}wrist_3_joint">
         <command_interface name="position"/>
-        <state_interface name="position"/>
+        <command_interface name="velocity"/>
+        <state_interface name="position">
+          <!-- initial position for the FakeSystem and simulation -->
+          <param name="initial_value">${initial_positions['wrist_3_joint']}</param>
+        </state_interface>
         <state_interface name="velocity"/>
-        <param name="min_position">-6.28318530718</param>
-        <param name="max_position">6.28318530718</param>
+        <state_interface name="effort"/>
       </joint>
     </ros2_control>

File: ur3_description/urdf/ur3.urdf.xacro (robot description, xacro)
@@ -60,5 +60,5 @@
    </xacro:ur_robot>
    <!-- call ur3 ros2_control macro -->
-   <xacro:ur3_ros2_control name="$(arg name)" prefix="$(arg prefix)"/>
+   <xacro:ur3_ros2_control name="$(arg name)" prefix="$(arg prefix)" initial_positions="${xacro.load_yaml(initial_positions_file)}"/>
    <!-- gazebo classic plugin -->
    <xacro:include filename="$(find ur3_description)/urdf/ur3.gazebo.xacro" />
